File: repro/repro.kicad_sch (KiCad schematic)
At the start: 1 part, among them U1 LK112M50TR

Commit message: Remove filter that causes the crash
Parts:
- U1: kicost.ldo.OPT_B:Foobar This filter field should cause the crash -> (none)
Changed lines of the file:
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@@
-      (effects (font (size 1.27 1.27)) hide)
-    )
-    (property "kicost.ldo.OPT_B:Foobar" "This filter field should cause the crash" (id 5) (at 157.48 81.28 0)
       (effects (font (size 1.27 1.27)) hide)
     )
